File: hardware/metallic_bear/metallic_bear.kicad_sch (KiCad schematic)
At the start: 18 parts, among them J1 MQ7_HEATER_SW, U1 W25Q128JVS

Commit message: add schema with kicad & lines
Parts:
- added J2: 5V_IN, Connector_PinHeader_2.54mm:PinHeader_1x02_P2.54mm_Vertical, symbol Connector_Generic:Conn_01x02
Connections:
- net +3V3: now also R4.2; no longer R4.1
- net +5V: now also A1.6 (E5V), J2.1 (Pin_1); no longer A1.18 (+5V)
- net GND: now also J2.2 (Pin_2)
- net I2C2_SCL: now also R4.1; no longer R4.2
- net MQ7_AO_5V: no longer names the net of A4.4 (AO), R6.1
Other:
- note added: "External 5 V supply feeds SCD30, the MQ7 heater board (J1) and the Nucleo (E5V) set the Nucleo 5V power-source jumper to E5V (see UM2505)"
- note added: "MQ7 module - AO to ADC1_IN1 (PA0) through R6/R7 (5 V max -> 3.2 V) Module VCC is the switched heater rail (5.0 V / 1.4 V) from the hardware/mq7_heater_switch board on J1, controlled by PC0 (MQ7_HEATER) J1: 1 +5V, 2 GND, 3 MQ7_HEATER, 4 MQ7_VCC - check pin order against that board"
- note added: "NUCLEO-G474RE (STM32G474RET6) ST morpho CN7 (left) / CN10 (right) Powered from the external 5 V supply through E5V (CN7-6)"
- note removed: "J1: to mq7_heater_switch board 1 +5V in, 2 GND, 3 MQ7_HEATER (PC0), 4 MQ7_VCC out (switched rail) check pin order against that board"
- note removed: "MQ7 module - AO to ADC1_IN1 (PA0) through a divider (5 V max -> 3.2 V) Module VCC is the switched heater rail (5.0 V / 1.4 V) from the hardware/mq7_heater_switch board, controlled by PC0 (MQ7_HEATER)"
- note removed: "NUCLEO-G474RE (STM32G474RET6) ST morpho CN7 (left) / CN10 (right) +3V3 and +5V come from the Nucleo"
